File: scheme-kicad5-120x180/g602.kicad_pcb (KiCad board)
At the start: 2 copper layers, 120 x 180 mm, 53 parts, among them Q1 IRL2203NPBF, Q2 IRL2203NPBF, U1 PC817, U2 PC817, U3 PC817, U4 PC817, U5 PC817, X3 arduino-nano, X4 TCST1103

Commit message: (refs scheme) Resisor updated.
Parts:
- R16: value 10 -> 60
Changed lines of the file:
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@@
       (effects (font (size 1 1) (thickness 0.15)))
     )
-    (fp_text value 10 (at 7.62 3.37 90) (layer F.Fab)
+    (fp_text value 60 (at 7.62 3.37 90) (layer F.Fab)
       (effects (font (size 1 1) (thickness 0.15)))
     )
